File: Design files/Behavioural board V2.brd (EAGLE design)
At the start: 92.4 x 94 mm, 49 parts, among them IC2 786TV, Q2 BSS138, Q3 BSS138, T1 BC337, T2 BC337, T3 BC337, T4 BC337

Commit message: v2
Connections:
- net ENC_A_3V3: now also U$1.23/A9; no longer U$1.13
Routing:
- net ENC_A_3V3: track 57.1 -> 94.6 mm
Changed lines of the file:
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@@
 <drawing>
 <settings>
-<setting alwaysvectorfont="yes"/>
+<setting alwaysvectorfont="no"/>
 <setting verticaltext="up"/>
 </settings>
@@
 <signal name="ENC_A_3V3">
 <contactref element="Q2" pad="2"/>
-<contactref element="U$1" pad="13"/>
 <contactref element="R17" pad="1"/>
 <wire x1="9.287" y1="63.566" x2="9.287" y2="63.185" width="0.4064" layer="1"/>
@@
 <via x="26.035" y="62.611" extent="1-16" drill="0.4064"/>
 <wire x1="26.035" y1="62.611" x2="27.686" y2="60.96" width="0.4064" layer="16"/>
-<wire x1="34.29" y1="44.577" x2="34.29" y2="40.513" width="0.4064" layer="16"/>
-<wire x1="34.29" y1="40.513" x2="35.433" y2="39.37" width="0.4064" layer="16"/>
-<wire x1="35.433" y1="39.37" x2="36.83" y2="39.37" width="0.4064" layer="16"/>
 <wire x1="17.907" y1="62.484" x2="18.542" y2="63.119" width="0.4064" layer="1"/>
 <wire x1="18.542" y1="63.119" x2="22.606" y2="63.119" width="0.4064" layer="1"/>
 <wire x1="22.606" y1="63.119" x2="23.114" y2="62.611" width="0.4064" layer="1"/>
 <wire x1="27.686" y1="60.96" x2="27.686" y2="51.181" width="0.4064" layer="16"/>
-<wire x1="27.686" y1="51.181" x2="34.29" y2="44.577" width="0.4064" layer="16"/>
+<wire x1="27.686" y1="51.181" x2="33.9725" y2="44.8945" width="0.4064" layer="16"/>
+<contactref element="U$1" pad="23/A9"/>
+<wire x1="33.9725" y1="44.8945" x2="33.9725" y2="36.5125" width="0.4064" layer="16"/>
+<wire x1="33.9725" y1="36.5125" x2="38.608" y2="31.877" width="0.4064" layer="16"/>
+<wire x1="38.608" y1="31.877" x2="60.452" y2="31.877" width="0.4064" layer="16"/>
+<wire x1="62.23" y1="33.655" x2="62.23" y2="39.37" width="0.4064" layer="16"/>
+<wire x1="60.452" y1="31.877" x2="62.23" y2="33.655" width="0.4064" layer="16"/>
 </signal>
 <signal name="ENC_B_3V3">
