File: Design files/Behavioural board V2.sch (EAGLE design)
At the start: 49 parts, among them IC2 786TV, T1 BC337, T2 BC337, T3 BC337, T4 BC337, X1 1-227161-0, X2 1-227161-0, X3 1-227161-0, X4 1-227161-0, X5 1-227161-0, X6 1-227161-0, X7 1-227161-0, X8 1-227161-0

Commit message: V2
Parts:
- removed 12V, GND, L1(1), L1(2), L2(1), L2(2), L3(1), L3(2), L4(1), L4(2): (no value), pinhead:PINHD-1X1
- removed TEENSYBOTTOM, TEENSYTOP: (no value), pinhead:PINHD-1X14
- removed TEENSYMIDDLE: (no value), pinhead:PINHD-1X5
- removed X1: 1-227161-0, con-coax_xavi:1-227161-0
- removed X2, X3, X4, X5, X6, X7, X8: 1-227161-0, con-coax:1-227161-0
- added DAC, LICK_1, LICK_2, LICK_3, LICK_4, TRIG_1, TRIG_2, TRIG_3, TRIG_4: 1-227161-0, con-coax_xavi:1-227161-0
- added J1: (no value), con-jack:JACK-PLUG0
- added JP1: (no value), pinhead:PINHD-1X5
- added Q2, Q3: BSS138, SparkFun:MOSFET-NCHANNELSMD
- added R13, R14, R15, R17: 10k, rcl:R-US_0207/10
- added VALVE_1, VALVE_2, VALVE_3, VALVE_4: (no value), pinhead:PINHD-1X2
Connections:
- removed net 5V: C2(0.1UF).1, D1.C, D2.C, D3.C, D4.C, IC2.VO, L1(2).1, L2(2).1, L3(2).1, L4(2).1, TEENSYBOTTOM.14
- removed net N$10: TEENSYTOP.6, X7.1
- removed net N$11: R3.2, TEENSYBOTTOM.5
- removed net N$12: R11.2, TEENSYTOP.14
- removed net N$13: R4.2, TEENSYBOTTOM.6
- removed net N$16: R5.2, TEENSYBOTTOM.7
- removed net N$17: R6.2, TEENSYBOTTOM.8
- removed net N$18: R7.2, TEENSYBOTTOM.9
- removed net N$19: R8.2, TEENSYBOTTOM.10
- removed net N$2: TEENSYTOP.4, X5.1
- removed net N$26: TEENSYBOTTOM.11, X8.1
- removed net N$27: R9.2, TEENSYTOP.13
- removed net N$3: TEENSYTOP.9, X2.1
- removed net N$30: R10.2, TEENSYTOP.12
- removed net N$36: R12.2, TEENSYTOP.11
- removed net N$37: C1(0.33UF).2, C2(0.1UF).2, GND.1, IC2.GND, T1.E, T2.E, T3.E, T4.E, TEENSYTOP.1, X1.2, X2.2, X3.2, X4.2, X5.2, X6.2, X7.2, X8.2
- removed net N$4: 12V.1, C1(0.33UF).1, IC2.VI
- removed net N$5: TEENSYTOP.7, X4.1
- removed net N$6: TEENSYTOP.8, X3.1
- removed net N$7: R1.2, TEENSYBOTTOM.3
- removed net N$8: TEENSYTOP.5, X6.1
- removed net N$9: R2.2, TEENSYBOTTOM.4
- new net 12V: C1(0.33UF).1, IC2.VI, J1.3
- new net CAP_IN_1: R2.2, U$1.16/A2/PWM/T
- new net CAP_IN_2: R4.2, U$1.18/A4/T/SDA
- new net CAP_IN_3: R6.2, U$1.20/A6/PWM/SCK1
- new net CAP_IN_4: R8.2, U$1.22/A8/T/PWM/SCL1
- new net CAP_OUT_1: R1.2, U$1.15/A1/T
- new net CAP_OUT_2: R3.2, U$1.17/A3/PWM/T
- new net CAP_OUT_3: R5.2, U$1.19/A5/T/SCL
- new net CAP_OUT_4: R7.2, U$1.21/A7
- new net ENC_A: JP1.4, Q2.D, R13.1
- new net ENC_A_3V3: Q2.S, R17.1, U$1.13/SCK/LED
- new net ENC_B: JP1.3, Q3.D, R15.1
- new net ENC_B_3V3: Q3.S, R14.1, U$1.14/A0
- new net GND: C1(0.33UF).2, C2(0.1UF).2, DAC.2, IC2.GND, J1.1, JP1.1, JP1.2, LICK_1.2, LICK_2.2, LICK_3.2, LICK_4.2, T1.E, T2.E, T3.E, T4.E, TRIG_1.2, TRIG_2.2, TRIG_3.2, TRIG_4.2, U$1.GND
- new net LICK_1: LICK_1.1, U$1.5
- new net LICK_2: LICK_2.1, U$1.6/PWM
- new net LICK_3: LICK_3.1, U$1.7/RX3
- new net LICK_4: LICK_4.1, U$1.8/TX3
- new net TRIG_1: TRIG_1.1, U$1.1/TX1/T/MISO1
- new net TRIG_2: TRIG_2.1, U$1.2
- new net TRIG_3: TRIG_3.1, U$1.3/T/PWM
- new net TRIG_4: TRIG_4.1, U$1.4/T/PWM
- new net VALVE_1: R11.2, U$1.12/MISO
- new net VALVE_2: R9.2, U$1.11/MOSI
- new net VALVE_3: R10.2, U$1.10/TX2/PWM
- new net VALVE_4: R12.2, U$1.9/RX2/PWM
- new net VCC: C2(0.1UF).1, D1.C, D2.C, D3.C, D4.C, IC2.VO, JP1.5, R13.2, R15.2, U$1.VIN, VALVE_1.2, VALVE_2.2, VALVE_3.2, VALVE_4.2
- new net VDD: Q2.G, Q3.G, R14.2, R17.2, U$1.3.3V
- net N$1: now also DAC.1, U$1.26/A12/DAC; no longer TEENSYTOP.10, X1.1
- net N$25: now also VALVE_1.1; no longer L1(1).1
- net N$29: now also VALVE_2.1; no longer L2(1).1
- net N$32: now also VALVE_3.1; no longer L3(1).1
- net N$35: now also VALVE_4.1; no longer L4(1).1
Other:
- note added: "Logic level shifter"
- moved on the sheet: C1(0.33UF), C2(0.1UF), CAPACITIVE1, CAPACITIVE2, CAPACITIVE3, CAPACITIVE4, D1, D2, D3, D4, IC2, R1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

Commit message: v2
Connections:
- net ENC_A_3V3: now also U$1.23/A9/T/PWM/SDA1; no longer U$1.13/SCK/LED
Changed lines of the file:
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@@
 <grid distance="1.27" unitdist="mm" unit="mm" style="lines" multiple="1" display="no" altdistance="0.01" altunitdist="inch" altunit="inch"/>
 <layers>
-<layer number="1" name="Top" color="4" fill="1" visible="yes" active="no"/>
-<layer number="2" name="Route2" color="1" fill="3" visible="yes" active="no"/>
-<layer number="3" name="Route3" color="4" fill="3" visible="yes" active="no"/>
-<layer number="4" name="Route4" color="1" fill="4" visible="yes" active="no"/>
-<layer number="5" name="Route5" color="4" fill="4" visible="yes" active="no"/>
-<layer number="6" name="Route6" color="1" fill="8" visible="yes" active="no"/>
-<layer number="7" name="Route7" color="4" fill="8" visible="yes" active="no"/>
-<layer number="8" name="Route8" color="1" fill="2" visible="yes" active="no"/>
-<layer number="9" name="Route9" color="4" fill="2" visible="yes" active="no"/>
-<layer number="10" name="Route10" color="1" fill="7" visible="yes" active="no"/>
-<layer number="11" name="Route11" color="4" fill="7" visible="yes" active="no"/>
-<layer number="12" name="Route12" color="1" fill="5" visible="yes" active="no"/>
-<layer number="13" name="Route13" color="4" fill="5" visible="yes" active="no"/>
-<layer number="14" name="Route14" color="1" fill="6" visible="yes" active="no"/>
-<layer number="15" name="Route15" color="4" fill="6" visible="yes" active="no"/>
-<layer number="16" name="Bottom" color="1" fill="1" visible="yes" active="no"/>
-<layer number="17" name="Pads" color="2" fill="1" visible="yes" active="no"/>
-<layer number="18" name="Vias" color="2" fill="1" visible="yes" active="no"/>
-<layer number="19" name="Unrouted" color="6" fill="1" visible="yes" active="no"/>
-<layer number="20" name="Dimension" color="24" fill="1" visible="yes" active="no"/>
-<layer number="21" name="tPlace" color="7" fill="1" visible="yes" active="no"/>
-<layer number="22" name="bPlace" color="7" fill="1" visible="yes" active="no"/>
-<layer number="23" name="tOrigins" color="15" fill="1" visible="yes" active="no"/>
-<layer number="24" name="bOrigins" color="15" fill="1" visible="yes" active="no"/>
-<layer number="25" name="tNames" color="7" fill="1" visible="yes" active="no"/>
-<layer number="26" name="bNames" color="7" fill="1" visible="yes" active="no"/>
-<layer number="27" name="tValues" color="7" fill="1" visible="yes" active="no"/>
-<layer number="28" name="bValues" color="7" fill="1" visible="yes" active="no"/>
+<layer number="1" name="Top" color="4" fill="1" visible="no" active="no"/>
+<layer number="2" name="Route2" color="1" fill="3" visible="no" active="no"/>
+<layer number="3" name="Route3" color="4" fill="3" visible="no" active="no"/>
+<layer number="4" name="Route4" color="1" fill="4" visible="no" active="no"/>
+<layer number="5" name="Route5" color="4" fill="4" visible="no" active="no"/>
+<layer number="6" name="Route6" color="1" fill="8" visible="no" active="no"/>
+<layer number="7" name="Route7" color="4" fill="8" visible="no" active="no"/>
+<layer number="8" name="Route8" color="1" fill="2" visible="no" active="no"/>
+<layer number="9" name="Route9" color="4" fill="2" visible="no" active="no"/>
+<layer number="10" name="Route10" color="1" fill="7" visible="no" active="no"/>
+<layer number="11" name="Route11" color="4" fill="7" visible="no" active="no"/>
+<layer number="12" name="Route12" color="1" fill="5" visible="no" active="no"/>
+<layer number="13" name="Route13" color="4" fill="5" visible="no" active="no"/>
+<layer number="14" name="Route14" color="1" fill="6" visible="no" active="no"/>
+<layer number="15" name="Route15" color="4" fill="6" visible="no" active="no"/>
+<layer number="16" name="Bottom" color="1" fill="1" visible="no" active="no"/>
+<layer number="17" name="Pads" color="2" fill="1" visible="no" active="no"/>
+<layer number="18" name="Vias" color="2" fill="1" visible="no" active="no"/>
+<layer number="19" name="Unrouted" color="6" fill="1" visible="no" active="no"/>
+<layer number="20" name="Dimension" color="24" fill="1" visible="no" active="no"/>
+<layer number="21" name="tPlace" color="7" fill="1" visible="no" active="no"/>
+<layer number="22" name="bPlace" color="7" fill="1" visible="no" active="no"/>
+<layer number="23" name="tOrigins" color="15" fill="1" visible="no" active="no"/>
+<layer number="24" name="bOrigins" color="15" fill="1" visible="no" active="no"/>
+<layer number="25" name="tNames" color="7" fill="1" visible="no" active="no"/>
+<layer number="26" name="bNames" color="7" fill="1" visible="no" active="no"/>
+<layer number="27" name="tValues" color="7" fill="1" visible="no" active="no"/>
+<layer number="28" name="bValues" color="7" fill="1" visible="no" active="no"/>
 <layer number="29" name="tStop" color="7" fill="3" visible="no" active="no"/>
 <layer number="30" name="bStop" color="7" fill="6" visible="no" active="no"/>
@@
 <layer number="35" name="tGlue" color="7" fill="4" visible="no" active="no"/>
 <layer number="36" name="bGlue" color="7" fill="5" visible="no" active="no"/>
-<layer number="37" name="tTest" color="7" fill="1" visible="yes" active="no"/>
-<layer number="38" name="bTest" color="7" fill="1" visible="yes" active="no"/>
+<layer number="37" name="tTest" color="7" fill="1" visible="no" active="no"/>
+<layer number="38" name="bTest" color="7" fill="1" visible="no" active="no"/>
 <layer number="39" name="tKeepout" color="4" fill="11" visible="no" active="no"/>
 <layer number="40" name="bKeepout" color="1" fill="11" visible="no" active="no"/>
@@
 <layer number="44" name="Drills" color="7" fill="1" visible="no" active="no"/>
 <layer number="45" name="Holes" color="7" fill="1" visible="no" active="no"/>
-<layer number="46" name="Milling" color="3" fill="1" visible="yes" active="no"/>
-<layer number="47" name="Measures" color="7" fill="1" visible="yes" active="no"/>
-<layer number="48" name="Document" color="7" fill="1" visible="yes" active="no"/>
-<layer number="49" name="Reference" color="7" fill="1" visible="yes" active="no"/>
-<layer number="50" name="dxf" color="12" fill="1" visible="yes" active="no"/>
-<layer number="51" name="tDocu" color="7" fill="1" visible="yes" active="no"/>
-<layer number="52" name="bDocu" color="7" fill="1" visible="yes" active="no"/>
-<layer number="53" name="tGND_GNDA" color="7" fill="1" visible="yes" active="no"/>
-<layer number="54" name="bGND_GNDA" color="7" fill="1" visible="yes" active="no"/>
-<layer number="56" name="wert" color="7" fill="1" visible="yes" active="no"/>
+<layer number="46" name="Milling" color="3" fill="1" visible="no" active="no"/>
+<layer number="47" name="Measures" color="7" fill="1" visible="no" active="no"/>
+<layer number="48" name="Document" color="7" fill="1" visible="no" active="no"/>
+<layer number="49" name="Reference" color="7" fill="1" visible="no" active="no"/>
+<layer number="50" name="dxf" color="12" fill="1" visible="no" active="no"/>
+<layer number="51" name="tDocu" color="7" fill="1" visible="no" active="no"/>
+<layer number="52" name="bDocu" color="7" fill="1" visible="no" active="no"/>
+<layer number="53" name="tGND_GNDA" color="7" fill="1" visible="no" active="no"/>
+<layer number="54" name="bGND_GNDA" color="7" fill="1" visible="no" active="no"/>
+<layer number="56" name="wert" color="7" fill="1" visible="no" active="no"/>
 <layer number="57" name="tCAD" color="7" fill="1" visible="no" active="no"/>
 <layer number="59" name="tCarbon" color="7" fill="1" visible="no" active="no"/>
@@
 </segment>
 <segment>
-<pinref part="U$1" gate="G$1" pin="13/SCK/LED"/>
-<wire x1="-269.24" y1="99.06" x2="-283.21" y2="99.06" width="0.1524" layer="91"/>
-<label x="-283.21" y="99.06" size="1.778" layer="95"/>
-</segment>
-</net>
+<pinref part="U$1" gate="G$1" pin="23/A9/T/PWM/SDA1"/>
+<wire x1="-269.24" y1="73.66" x2="-283.21" y2="73.66" width="0.1524" layer="91"/>
+<label x="-283.21" y="73.66" size="1.778" layer="95"/>
+</segment>
+</net>
